Commit message: Modifying launch files

File: catkin_ws/src/sigsent/urdf/hokuyo.urdf.xacro (robot description, xacro)
@@ -56,5 +56,5 @@
             <plugin name="gazebo_ros_head_hokuyo_controller" filename="libgazebo_ros_laser.so">
                 <robotNamespace></robotNamespace>
-                <topicName>laser_scan</topicName>
+                <topicName>/scan</topicName>
                 <frameName>hokuyo_laser_link</frameName>
             </plugin>

File: catkin_ws/src/sigsent/urdf/kobuki.urdf.xacro (robot description, xacro)
@@ -10,6 +10,10 @@
 <xacro:include filename="$(find turtlebot_description)/urdf/stacks/hexagons.urdf.xacro"/>
 <xacro:include filename="$(find sigsent)/urdf/hokuyo.urdf.xacro"/>
+<xacro:include filename="$(find hector_sensors_description)/urdf/hokuyo_utm30lx.urdf.xacro"/>
 <kobuki/>
-	<stack_hexagons parent="base_link"/>
-	<sensor_kinect  parent="base_link"/>
+<stack_hexagons parent="base_link"/>
+<sensor_kinect  parent="base_link"/>
+<hokuyo_utm30lx_model name="hokuyo_laser" parent="base_link">
+    <origin xyz="0 0 +0.30" rpy="0 0 0" />
+</hokuyo_utm30lx_model>
 </robot>
