Commit message: Laserscan working :)

File: catkin_ws/src/sigsent/urdf/kobuki.urdf.xacro (robot description, xacro)
@@ -9,11 +9,10 @@
 <xacro:include filename="$(find kobuki_description)/urdf/kobuki.urdf.xacro" />
 <xacro:include filename="$(find turtlebot_description)/urdf/stacks/hexagons.urdf.xacro"/>
-<xacro:include filename="$(find sigsent)/urdf/hokuyo.urdf.xacro"/>
-<xacro:include filename="$(find hector_sensors_description)/urdf/hokuyo_utm30lx.urdf.xacro"/>
 <kobuki/>
 <stack_hexagons parent="base_link"/>
 <sensor_kinect  parent="base_link"/>
-<hokuyo_utm30lx_model name="hokuyo_laser" parent="base_link">
-    <origin xyz="0 0 +0.30" rpy="0 0 0" />
-</hokuyo_utm30lx_model>
+<xacro:include filename="$(find hector_sensors_description)/urdf/hokuyo_utm30lx.urdf.xacro"/>
+<xacro:hokuyo_utm30lx name="hokuyo_laser" parent="base_link" ros_topic="scan" update_rate="40" ray_count="1081" min_angle="135" max_angle="-135">
+    <origin xyz="0 0 +0.45" rpy="0 0 0" />
+</xacro:hokuyo_utm30lx>
 </robot>

Commit message: Adding camera in progress

File: catkin_ws/src/sigsent/urdf/kobuki.urdf.xacro (robot description, xacro)
@@ -12,4 +12,8 @@
 <stack_hexagons parent="base_link"/>
 <sensor_kinect  parent="base_link"/>
+<xacro:include filename="$(find hector_sensors_description)/urdf/generic_camera.urdf.xacro"/>
+<xacro:generic_camera name="cam1" ros_topic="image_raw" cam_info_topic="camera_info" parent="base_link" update_rate="60" res_x="640" res_y="360" image_format="R8G8B8" hfov="90">
+  <origin xyz="0 0 +0.5" rpy="0 0 0"/>
+</xacro:generic_camera>
 <xacro:include filename="$(find hector_sensors_description)/urdf/hokuyo_utm30lx.urdf.xacro"/>
 <xacro:hokuyo_utm30lx name="hokuyo_laser" parent="base_link" ros_topic="scan" update_rate="40" ray_count="1081" min_angle="135" max_angle="-135">
